File: Cafebabe/Schematics/SD-SAO/SDtoSAOadapter.kicad_sch (KiCad schematic)
At the start: 2 parts

Commit message: V1 Cafebabe firmware complete
Parts:
- gave numbers to parts that had none: 2
Changed lines of the file:
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@@
   (symbol (lib_id "power:VCC") (at 137.16 73.66 270) (unit 1)
     (in_bom yes) (on_board yes)
-    (property "Reference" "#PWR?" (id 0) (at 133.35 73.66 0)
+    (property "Reference" "#PWR0104" (id 0) (at 133.35 73.66 0)
       (effects (font (size 1.27 1.27)) hide)
     )
@@
   (symbol (lib_id "power:VSS") (at 137.16 78.74 270) (unit 1)
     (in_bom yes) (on_board yes)
-    (property "Reference" "#PWR?" (id 0) (at 133.35 78.74 0)
+    (property "Reference" "#PWR0103" (id 0) (at 133.35 78.74 0)
       (effects (font (size 1.27 1.27)) hide)
     )
@@
   (symbol (lib_id "power:VCC") (at 194.31 66.04 0) (unit 1)
     (in_bom yes) (on_board yes)
-    (property "Reference" "#PWR?" (id 0) (at 194.31 69.85 0)
+    (property "Reference" "#PWR0102" (id 0) (at 194.31 69.85 0)
       (effects (font (size 1.27 1.27)) hide)
     )
@@
   (symbol (lib_id "power:VSS") (at 194.31 81.28 180) (unit 1)
     (in_bom yes) (on_board yes)
-    (property "Reference" "#PWR?" (id 0) (at 194.31 77.47 0)
+    (property "Reference" "#PWR0101" (id 0) (at 194.31 77.47 0)
       (effects (font (size 1.27 1.27)) hide)
     )
@@
   (symbol (lib_id "Connector_Generic:Conn_02x03_Odd_Even") (at 191.77 72.39 270) (unit 1)
     (in_bom yes) (on_board yes)
-    (property "Reference" "J?" (id 0) (at 199.8218 73.66 0))
+    (property "Reference" "J2" (id 0) (at 199.8218 73.66 0))
     (property "Value" "Conn_02x03_Odd_Even" (id 1) (at 197.5104 73.66 0))
     (property "Footprint" "Connector_PinHeader_2.54mm:PinHeader_2x03_P2.54mm_Vertical" (id 2) (at 191.77 72.39 0)
@@
   (symbol (lib_id "Connector:Micro_SD_Card") (at 113.03 73.66 0) (mirror y) (unit 1)
     (in_bom yes) (on_board yes)
-    (property "Reference" "J?" (id 0) (at 114.3 55.4482 0))
+    (property "Reference" "J1" (id 0) (at 114.3 55.4482 0))
     (property "Value" "Micro_SD_Card" (id 1) (at 114.3 57.7596 0))
     (property "Footprint" "Voltlog:microSD_card" (id 2) (at 83.82 66.04 0)
@@
   )
   (symbol_instances
+    (path "/ab32b0b8-f7ed-4515-b6ff-a1bced9f4ca2"
+      (reference "#PWR0101") (unit 1) (value "VSS") (footprint "")
+    )
     (path "/75cf8a15-fae0-4ad2-af87-43af1d71d09a"
-      (reference "#PWR?") (unit 1) (value "VCC") (footprint "")
-    )
-    (path "/ab32b0b8-f7ed-4515-b6ff-a1bced9f4ca2"
-      (reference "#PWR?") (unit 1) (value "VSS") (footprint "")
+      (reference "#PWR0102") (unit 1) (value "VCC") (footprint "")
     )
     (path "/b1bd2a49-1c56-4b4e-9b8b-f2eba55cd279"
-      (reference "#PWR?") (unit 1) (value "VSS") (footprint "")
+      (reference "#PWR0103") (unit 1) (value "VSS") (footprint "")
     )
     (path "/b356a5a0-4cdb-4838-bf39-467015a12562"
-      (reference "#PWR?") (unit 1) (value "VCC") (footprint "")
+      (reference "#PWR0104") (unit 1) (value "VCC") (footprint "")
     )
     (path "/1de83ced-efc6-4cdb-aba2-bc3322e0f053"
-      (reference "J?") (unit 1) (value "Micro_SD_Card") (footprint "Voltlog:microSD_card")
+      (reference "J1") (unit 1) (value "Micro_SD_Card") (footprint "Voltlog:microSD_card")
     )
     (path "/91b82d1a-32ca-41ff-b297-05fea20bde2b"
-      (reference "J?") (unit 1) (value "Conn_02x03_Odd_Even") (footprint "Connector_PinHeader_2.54mm:PinHeader_2x03_P2.54mm_Vertical")
+      (reference "J2") (unit 1) (value "Conn_02x03_Odd_Even") (footprint "Connector_PinHeader_2.54mm:PinHeader_2x03_P2.54mm_Vertical")
     )
   )
