File: TouchSplit/Schematics/Left/TouchSplitLeft.kicad_sch (KiCad schematic)
At the start: 82 parts

Commit message: Updating for hondouras trip
Parts:
- removed J?: Conn_01x11, symbol Connector_Generic:Conn_01x11
- added BT1: Battery_Cell, Tests:Dongguan14500, symbol Device:Battery_Cell
- added C17: 10uF, Capacitor_SMD:C_0805_2012Metric, symbol Device:C_Small
- added C18, C19: 1uF, Capacitor_SMD:C_0805_2012Metric, symbol Device:C
- added D4: LED_Small, LED_SMD:LED_0805_2012Metric, symbol Device:LED_Small
- added J1: Conn_01x07, Connector_PinHeader_2.54mm:PinHeader_1x07_P2.54mm_Vertical, symbol Connector_Generic:Conn_01x07
- added Power->1: SW3, BreadBoardPwr:SK-3296S_switch, symbol Switch:SW_SPDT
- added R13: 1k, Resistor_SMD:R_0805_2012Metric, symbol Device:R_Small
- added R14: Charger Bypass, Resistor_SMD:R_0805_2012Metric, symbol Device:R_Small
- added R15: 2.5k, Resistor_SMD:R_0805_2012Metric, symbol Device:R_Small
- added RN8: R_Pack04, Resistor_SMD:R_Array_Convex_4x0603, symbol Device:R_Pack04
- added U5: HX4055M, Package_TO_SOT_SMD:SOT-23-5, symbol TwitterKeyboard-rescue:HX4055M-MechKeyboard
- added U6: TLV1117-33, Package_TO_SOT_SMD:SOT-223-3_TabPin2, symbol Regulator_Linear:TLV1117-33
- C1, C10, C11, C12, C13, C14, C15, C16, C2, C5, C6, C7, C8, C9: renamed from C?; footprint (none) -> Capacitor_SMD:C_0805_2012Metric
- D1, D2, D3: renamed from D?; footprint (none) -> LED_SMD:LED_0805_2012Metric
- J10, J11, J12, J13, J15, J16, J17, J18, J19, J2, J20, J21, J22, J23, J24, J25, J26, J27, J28, J29, J3, J30, J31, J32, J33, J34, J35, J4, J5, J6, J7, J8, J9: renamed from J?; footprint (none) -> TouchSplit:Pad
- J14: renamed from J?; footprint (none) -> Connector_PinHeader_2.54mm:PinHeader_1x04_P2.54mm_Vertical
- R1, R10, R11, R12, R2, R3, R4, R5, R6, R7, R8, R9: renamed from R?; footprint (none) -> Resistor_SMD:R_0805_2012Metric
- RN1, RN10, RN2, RN3, RN5, RN6, RN7, RN9: renamed from RN?; footprint (none) -> Resistor_SMD:R_Array_Convex_4x0603
- U3: renamed from U?; footprint (none) -> TouchSplit:ESP32-C3-Mini-1
- gave numbers to parts that had none: 9
Connections:
- net IO6 is gone; now on net ADC1: U3.20 (IO6)
- net IO7 is gone; now on net ADC2: U3.21 (IO7)
- net SCL is gone; now on net IO5: U1.21 (SCL), U2.21 (SCL), U4.14 (SCL)
- net SDA is gone; now on net IO4: U1.22 (SDA), U2.22 (SDA), U4.15 (SDA)
- net IO0: now also J1.1 (Pin_1)
- net IO1: now also J1.2 (Pin_2)
- net IO10: now also J1.7 (Pin_7)
- net IO2: now also J1.3 (Pin_3)
- net IO3: now also J1.4 (Pin_4)
- net IO4: now also RN8.2 (R2.1)
- net IO5: now also RN8.1 (R1.1)
- net IO8: now also J1.5 (Pin_5)
- net IO9: now also J1.6 (Pin_6)
- net VBUS: now also R13.2, R14.1, U5.4 (VCC)
- net VCC: now also C19.1, RN8.7 (R2.2), RN8.8 (R1.2), U6.2 (VO)
- net VSS: now also BT1.2 (-), C17.2, C18.2, C19.2, R15.1, U5.2 (Gnd), U6.1 (GND)
- new net: D4.1 (K), U5.1 (Chrg)
- new net: R15.2, U5.5 (PROG)
- new net: D4.2 (A), R13.1
- new net: C18.1, Power->1.2 (B), U6.3 (VI)
- new net VDDA: BT1.1 (+), C17.1, Power->1.3 (C), R14.2, U5.3 (Bat)
- no-connect marks 21 -> 26
Other:
- moved on the sheet: C12, C13, C3, C4, J14, P1, RN4
